File: _autosave-Grid Selector.kicad_sch (KiCad schematic)
At the start: 122 parts, among them SW1 MX_SW_HS, SW10 MX_SW_HS, SW11 MX_SW_HS, SW12 MX_SW_HS, SW13 MX_SW_HS, SW14 MX_SW_HS, SW15 MX_SW_HS, SW16 MX_SW_HS, SW17 MX_SW_HS, SW18 MX_SW_HS, SW19 MX_SW_HS, SW2 MX_SW_HS, SW20 MX_SW_HS, SW21 MX_SW_HS, SW22 MX_SW_HS, SW23 MX_SW_HS, SW24 MX_SW_HS, SW25 MX_SW_HS, SW26 MX_SW_HS, SW27 MX_SW_HS, SW28 MX_SW_HS, SW29 MX_SW_HS, SW3 MX_SW_HS, SW30 MX_SW_HS, SW4 MX_SW_HS, SW5 MX_SW_HS, SW6 MX_SW_HS, SW7 MX_SW_HS, SW8 MX_SW_HS, SW9 MX_SW_HS, U1 Pico

Commit message: routed oled
Connections:
- net COL0: now also U1.12 (GPIO9); no longer U1.15 (GPIO11)
- net COL1: now also U1.11 (GPIO8); no longer U1.12 (GPIO9)
- net COL2: now also U1.10 (GPIO7); no longer U1.11 (GPIO8)
- net COL3: now also U1.9 (GPIO6); no longer U1.10 (GPIO7)
- net COL4: now also U1.7 (GPIO5); no longer U1.9 (GPIO6)
- net COL5: now also U1.6 (GPIO4); no longer U1.7 (GPIO5)
- net COL6: now also U1.5 (GPIO3); no longer U1.6 (GPIO4)
- net GND: now also U1.18 (GND); no longer U1.8 (GND)
- net ROW0: now also U1.15 (GPIO11); no longer U1.5 (GPIO3)
- net ROW1: now also U1.16 (GPIO12); no longer U1.14 (GPIO10)
- net ROW2: now also U1.17 (GPIO13); no longer U1.20 (GPIO15)
- net LEDIN: now reaches LED1.3 (DIN)
Changed lines of the file:
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@@
     (stroke (width 0) (type default) (color 0 0 0 0))
   )
-  (wire (pts (xy 181.61 47.625) (xy 191.135 47.625))
+  (wire (pts (xy 181.61 73.025) (xy 191.135 73.025))
     (stroke (width 0) (type default) (color 0 0 0 0))
   )
@@
     (stroke (width 0) (type default) (color 0 0 0 0))
   )
-  (global_label "COL5" (shape input) (at 191.135 45.085 180) (fields_autoplaced)
-    (effects (font (size 1.27 1.27)) (justify right))
-    (property "Intersheet References" "${INTERSHEET_REFS}" (id 0) (at 183.8838 45.0056 0)
+  (global_label "COL5" (shape input) (at 191.135 42.545 180) (fields_autoplaced)
+    (effects (font (size 1.27 1.27)) (justify right))
+    (property "Intersheet References" "${INTERSHEET_REFS}" (id 0) (at 183.8838 42.4656 0)
       (effects (font (size 1.27 1.27)) (justify right) hide)
     )
@@
     )
   )
-  (global_label "COL1" (shape input) (at 191.135 57.785 180) (fields_autoplaced)
-    (effects (font (size 1.27 1.27)) (justify right))
-    (property "Intersheet References" "${INTERSHEET_REFS}" (id 0) (at 183.8838 57.7056 0)
+  (global_label "COL1" (shape input) (at 191.135 55.245 180) (fields_autoplaced)
+    (effects (font (size 1.27 1.27)) (justify right))
+    (property "Intersheet References" "${INTERSHEET_REFS}" (id 0) (at 183.8838 55.1656 0)
       (effects (font (size 1.27 1.27)) (justify right) hide)
     )
@@
     )
   )
-  (global_label "COL3" (shape input) (at 191.135 52.705 180) (fields_autoplaced)
-    (effects (font (size 1.27 1.27)) (justify right))
-    (property "Intersheet References" "${INTERSHEET_REFS}" (id 0) (at 183.8838 52.6256 0)
+  (global_label "COL3" (shape input) (at 191.135 50.165 180) (fields_autoplaced)
+    (effects (font (size 1.27 1.27)) (justify right))
+    (property "Intersheet References" "${INTERSHEET_REFS}" (id 0) (at 183.8838 50.0856 0)
+      (effects (font (size 1.27 1.27)) (justify right) hide)
+    )
+  )
+  (global_label "LEDIN" (shape input) (at 19.685 102.87 180) (fields_autoplaced)
+    (effects (font (size 1.27 1.27)) (justify right))
+    (property "Intersheet References" "${INTERSHEET_REFS}" (id 0) (at 11.8895 102.7906 0)
       (effects (font (size 1.27 1.27)) (justify right) hide)
     )
@@
     )
   )
-  (global_label "COL2" (shape input) (at 191.135 55.245 180) (fields_autoplaced)
-    (effects (font (size 1.27 1.27)) (justify right))
-    (property "Intersheet References" "${INTERSHEET_REFS}" (id 0) (at 183.8838 55.1656 0)
+  (global_label "COL2" (shape input) (at 191.135 52.705 180) (fields_autoplaced)
+    (effects (font (size 1.27 1.27)) (justify right))
+    (property "Intersheet References" "${INTERSHEET_REFS}" (id 0) (at 183.8838 52.6256 0)
       (effects (font (size 1.27 1.27)) (justify right) hide)
     )
@@
     )
   )
-  (global_label "ROW2" (shape input) (at 191.135 78.105 180) (fields_autoplaced)
-    (effects (font (size 1.27 1.27)) (justify right))
-    (property "Intersheet References" "${INTERSHEET_REFS}" (id 0) (at 183.4605 78.0256 0)
+  (global_label "ROW2" (shape input) (at 191.135 70.485 180) (fields_autoplaced)
+    (effects (font (size 1.27 1.27)) (justify right))
+    (property "Intersheet References" "${INTERSHEET_REFS}" (id 0) (at 183.4605 70.4056 0)
       (effects (font (size 1.27 1.27)) (justify right) hide)
     )
@@
     )
   )
-  (global_label "COL4" (shape input) (at 191.135 50.165 180) (fields_autoplaced)
-    (effects (font (size 1.27 1.27)) (justify right))
-    (property "Intersheet References" "${INTERSHEET_REFS}" (id 0) (at 183.8838 50.0856 0)
-      (effects (font (size 1.27 1.27)) (justify right) hide)
-    )
-  )
-  (global_label "COL6" (shape input) (at 191.135 42.545 180) (fields_autoplaced)
-    (effects (font (size 1.27 1.27)) (justify right))
-    (property "Intersheet References" "${INTERSHEET_REFS}" (id 0) (at 183.8838 42.4656 0)
+  (global_label "COL4" (shape input) (at 191.135 45.085 180) (fields_autoplaced)
+    (effects (font (size 1.27 1.27)) (justify right))
+    (property "Intersheet References" "${INTERSHEET_REFS}" (id 0) (at 183.8838 45.0056 0)
+      (effects (font (size 1.27 1.27)) (justify right) hide)
+    )
+  )
+  (global_label "COL6" (shape input) (at 191.135 40.005 180) (fields_autoplaced)
+    (effects (font (size 1.27 1.27)) (justify right))
+    (property "Intersheet References" "${INTERSHEET_REFS}" (id 0) (at 183.8838 39.9256 0)
       (effects (font (size 1.27 1.27)) (justify right) hide)
     )
@@
     )
   )
-  (global_label "ROW0" (shape input) (at 191.135 40.005 180) (fields_autoplaced)
-    (effects (font (size 1.27 1.27)) (justify right))
-    (property "Intersheet References" "${INTERSHEET_REFS}" (id 0) (at 183.4605 39.9256 0)
-      (effects (font (size 1.27 1.27)) (justify right) hide)
-    )
-  )
-  (global_label "ROW1" (shape input) (at 191.135 62.865 180) (fields_autoplaced)
-    (effects (font (size 1.27 1.27)) (justify right))
-    (property "Intersheet References" "${INTERSHEET_REFS}" (id 0) (at 183.4605 62.7856 0)
+  (global_label "ROW0" (shape input) (at 191.135 65.405 180) (fields_autoplaced)
+    (effects (font (size 1.27 1.27)) (justify right))
+    (property "Intersheet References" "${INTERSHEET_REFS}" (id 0) (at 183.4605 65.3256 0)
+      (effects (font (size 1.27 1.27)) (justify right) hide)
+    )
+  )
+  (global_label "ROW1" (shape input) (at 191.135 67.945 180) (fields_autoplaced)
+    (effects (font (size 1.27 1.27)) (justify right))
+    (property "Intersheet References" "${INTERSHEET_REFS}" (id 0) (at 183.4605 67.8656 0)
       (effects (font (size 1.27 1.27)) (justify right) hide)
     )
@@
     )
   )
-  (global_label "COL0" (shape input) (at 191.135 65.405 180) (fields_autoplaced)
-    (effects (font (size 1.27 1.27)) (justify right))
-    (property "Intersheet References" "${INTERSHEET_REFS}" (id 0) (at 183.8838 65.3256 0)
+  (global_label "COL0" (shape input) (at 191.135 57.785 180) (fields_autoplaced)
+    (effects (font (size 1.27 1.27)) (justify right))
+    (property "Intersheet References" "${INTERSHEET_REFS}" (id 0) (at 183.8838 57.7056 0)
       (effects (font (size 1.27 1.27)) (justify right) hide)
     )
@@
     (pin "2")
   )
-  (symbol (lib_id "power:GND") (at 181.61 47.625 0) (unit 1)
-    (in_bom yes) (on_board yes) (fields_autoplaced)
-    (property "Reference" "#PWR0101" (id 0) (at 181.61 53.975 0)
-      (effects (font (size 1.27 1.27)) hide)
-    )
-    (property "Value" "GND" (id 1) (at 181.61 52.07 0))
-    (property "Footprint" "" (id 2) (at 181.61 47.625 0)
-      (effects (font (size 1.27 1.27)) hide)
-    )
-    (property "Datasheet" "" (id 3) (at 181.61 47.625 0)
-      (effects (font (size 1.27 1.27)) hide)
-    )
+  (symbol (lib_id "power:GND") (at 181.61 73.025 0) (unit 1)
+    (in_bom yes) (on_board yes) (fields_autoplaced)
+    (property "Reference" "#PWR0101" (id 0) (at 181.61 79.375 0)
+      (effects (font (size 1.27 1.27)) hide)
+    )
+    (property "Value" "GND" (id 1) (at 181.61 77.47 0))
+    (property "Footprint" "" (id 2) (at 181.61 73.025 0)
+      (effects (font (size 1.27 1.27)) hide)
+    )
+    (property "Datasheet" "" (id 3) (at 181.61 73.025 0)
+      (effects (font (size 1.27 1.27)) hide)
+    )
