File: _autosave-Grid Selector.kicad_pcb (KiCad board)
At the start: 2 copper layers, 235.6 x 60.3 mm, 122 parts, among them SW1 MX_SW_HS, SW10 MX_SW_HS, SW11 MX_SW_HS, SW12 MX_SW_HS, SW13 MX_SW_HS, SW14 MX_SW_HS, SW15 MX_SW_HS, SW16 MX_SW_HS, SW17 MX_SW_HS, SW18 MX_SW_HS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

Commit message: added logos
Parts:
- added G***: LOGO, LOGO, F.Cu at (64.8, 82.2)
- added G***: LOGO, logos:bureddo30, F.Cu at (65.9, 98.4)
