File: Grid Selector.kicad_pcb (KiCad board)
At the start: 2 copper layers, 235.6 x 60.3 mm, 122 parts, among them SW1 MX_SW_HS, SW10 MX_SW_HS, SW11 MX_SW_HS, SW12 MX_SW_HS, SW13 MX_SW_HS, SW14 MX_SW_HS, SW15 MX_SW_HS, SW16 MX_SW_HS, SW17 MX_SW_HS, SW18 MX_SW_HS, SW19 MX_SW_HS, SW2 MX_SW_HS, SW20 MX_SW_HS, SW21 MX_SW_HS, SW22 MX_SW_HS, SW23 MX_SW_HS, SW24 MX_SW_HS, SW25 MX_SW_HS, SW26 MX_SW_HS, SW27 MX_SW_HS, SW28 MX_SW_HS, SW29 MX_SW_HS, SW3 MX_SW_HS, SW30 MX_SW_HS, SW4 MX_SW_HS, SW5 MX_SW_HS, SW6 MX_SW_HS, SW7 MX_SW_HS, SW8 MX_SW_HS, SW9 MX_SW_HS, U1 Pico

Commit message: created gerber file
Parts:
- added G***: LOGO, logos:bureddo30, F.Cu at (58.5, 97.2)
- added G***: LOGO, LOGO, F.Cu at (64.8, 82.2)
Other:
- board text added: "designed by k hirota"

Commit message: reduced the size to 15 keys
Parts:
- removed D16, D17, D18, D19, D20, D21, D22, D23, D24, D25, D26, D27, D28, D29, D30: D_Small, Diode_SMD:D_SOD-123
- removed the G*** at (58.5, 97.2)
- removed the G*** at (64.8, 82.2)
- removed LED16, LED17, LED18, LED19, LED20, LED21, LED22, LED23, LED24, LED25, LED26, LED27, LED28, LED29, LED30: SK6812MINI-E, marbastlib-various:LED_6028R
- removed R16, R17, R18, R19, R20, R21, R22, R23, R24, R25, R26, R27, R28, R29, R30: 100 ohm, Resistor_SMD:R_0805_2012Metric
- removed SW16, SW17, SW18, SW19, SW20, SW21, SW22, SW23, SW24, SW25, SW26, SW27, SW28, SW29, SW30: MX_SW_HS, marbastlib-mx:SW_MX_HS_1u
- added G***: LOGO, logos:new5940logo, F.Cu at (157.6, 47.2)
- added G***: LOGO, logos:bureddo15, F.Cu at (158.3, 56.9)
- U1: moved to F.Cu
- moved OL1 115.5 mm to (162.5, 66.8), turned to 90 degrees
- moved D10 109.7 mm to (140.2, 159.3)
- moved LED10 109.7 mm to (132.3, 165.2)
- moved R10 109.7 mm to (132.3, 168.4)
- moved SW10 109.7 mm to (132.3, 160.1)
- moved D5 88.7 mm to (121.2, 159.3)
- moved LED5 88.7 mm to (113.2, 165.2)
- moved R4 88.7 mm to (113.2, 149.3)
- moved SW4 88.7 mm to (113.2, 141.0)
- moved D4 88.7 mm to (121.2, 140.2)
- moved LED4 88.7 mm to (113.2, 146.2)
- moved R5 88.7 mm to (113.2, 168.4)
- moved SW5 88.7 mm to (113.2, 160.1)
- moved D13 72.7 mm to (159.3, 121.2)
- moved D15 72.7 mm to (159.3, 159.3)
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Connections:
- D10 pad 1: ROW0 -> ROW4
- D11 pad 1: ROW1 -> ROW0
- D12 pad 1: ROW2 -> ROW1
- D13 pad 1: ROW0 -> ROW2
- D14 pad 1: ROW1 -> ROW3
- D15 pad 1: ROW2 -> ROW4
- D4 pad 1: ROW0 -> ROW3
- D5 pad 1: ROW1 -> ROW4
- D6 pad 1: ROW2 -> ROW0
- D7 pad 1: ROW0 -> ROW1
- D8 pad 1: ROW1 -> ROW2
- D9 pad 1: ROW2 -> ROW3
- LED10 pad 2: Net-(LED10-Pad2) -> Net-(LED15-Pad3)
- LED10 pad 3: Net-(LED10-Pad3) -> Net-(LED5-Pad2)
- LED13 pad 3: Net-(LED10-Pad2) -> Net-(LED8-Pad2)
- LED14 pad 3: Net-(LED11-Pad2) -> Net-(LED9-Pad2)
- LED15 pad 2: Net-(LED15-Pad2) -> unconnected-(LED15-Pad2)
- LED15 pad 3: Net-(LED12-Pad2) -> Net-(LED15-Pad3)
- LED2 pad 2: Net-(LED2-Pad2) -> Net-(LED7-Pad3)
- LED2 pad 3: Net-(LED2-Pad3) -> Net-(LED11-Pad2)
- LED3 pad 2: Net-(LED3-Pad2) -> Net-(LED8-Pad3)
- LED3 pad 3: Net-(LED29-Pad2) -> Net-(LED12-Pad2)
- LED4 pad 2: Net-(LED4-Pad2) -> Net-(LED9-Pad3)
- LED4 pad 3: Net-(LED1-Pad2) -> Net-(LED13-Pad2)
- LED5 pad 3: Net-(LED2-Pad2) -> Net-(LED14-Pad2)
- LED6 pad 2: Net-(LED6-Pad2) -> Net-(LED11-Pad3)
- LED6 pad 3: Net-(LED3-Pad2) -> Net-(LED1-Pad2)
- LED7 pad 2: Net-(LED10-Pad3) -> Net-(LED12-Pad3)
- LED7 pad 3: Net-(LED4-Pad2) -> Net-(LED7-Pad3)
- LED8 pad 2: Net-(LED11-Pad3) -> Net-(LED8-Pad2)
- LED8 pad 3: Net-(LED5-Pad2) -> Net-(LED8-Pad3)
- LED9 pad 2: Net-(LED12-Pad3) -> Net-(LED9-Pad2)
- LED9 pad 3: Net-(LED6-Pad2) -> Net-(LED9-Pad3)
- SW10 pad 1: COL3 -> COL1
- SW11 pad 1: COL3 -> COL2
- SW12 pad 1: COL3 -> COL2
- SW13 pad 1: COL4 -> COL2
- SW14 pad 1: COL4 -> COL2
- SW15 pad 1: COL4 -> COL2
- SW4 pad 1: COL1 -> COL0
- SW5 pad 1: COL1 -> COL0
- SW7 pad 1: COL2 -> COL1
- SW8 pad 1: COL2 -> COL1
- SW9 pad 1: COL2 -> COL1
- U1 pad 1: COL9 -> unconnected-(U1-Pad1)
- U1 pad 10: COL2 -> COL0
- U1 pad 12: COL0 -> unconnected-(U1-Pad12)
- U1 pad 14: LED -> unconnected-(U1-Pad14)
- U1 pad 15: ROW0 -> unconnected-(U1-Pad15)
- U1 pad 16: ROW1 -> unconnected-(U1-Pad16)
- U1 pad 17: ROW2 -> COL2
- U1 pad 2: COL8 -> ROW4
- U1 pad 25: unconnected-(U1-Pad25) -> SCL
- U1 pad 26: unconnected-(U1-Pad26) -> SDA
- U1 pad 31: SDA -> unconnected-(U1-Pad31)
- U1 pad 32: SCL -> unconnected-(U1-Pad32)
- U1 pad 33: GND -> unconnected-(U1-Pad33)
- U1 pad 4: COL7 -> ROW3
- U1 pad 5: COL6 -> ROW2
- U1 pad 6: COL5 -> ROW1
- U1 pad 7: COL4 -> LED
- U1 pad 9: COL3 -> ROW0
Routing:
- net GND: track 686.2 -> 412.4 mm, vias 4 -> 0
- net +5V: track 743.5 -> 479.8 mm, vias 11 -> 5
- net COL9: track 230.2 -> 0.00 mm, vias 4 -> 0
- net Net-(LED2-Pad3): track 214.2 -> 0.00 mm
- net Net-(LED29-Pad2): track 214.2 -> 0.00 mm
- net COL8: track 211.9 -> 0.00 mm, vias 4 -> 0
- net COL7: track 194.9 -> 0.00 mm, vias 4 -> 0
- net COL6: track 177.6 -> 0.00 mm, vias 4 -> 0
- net COL5: track 160.4 -> 0.00 mm, vias 4 -> 0
- net ROW4: track 0.00 -> 154.9 mm, vias 0 -> 1
- net COL4: track 150.1 -> 0.00 mm, vias 4 -> 0
- net ROW0: track 236.0 -> 89.2 mm, vias 2 -> 0
- net ROW3: track 0.00 -> 136.9 mm, vias 0 -> 1
- net COL3: track 128.4 -> 0.00 mm, vias 4 -> 0
- net ROW1: track 219.1 -> 101.9 mm
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Other:
- board size 235.6 x 60.3 mm -> 69.9 x 142.1 mm
- board text added: "designed by khirota"
- board text removed: "designed by k hirota"
